File: life-bms/helios-bms-life.kicad_sch (KiCad schematic)
At the start: 57 parts, among them J1 Outboard, J2 Debug, J3 Output, J4 Battery, Q1 SSM6J507NU, Q2 Q_Dual_NMOS_PMOS_S1G1D2S2G2D1, Q3 PMOS, U1 TPSM861253, U2 BQ25306, U3 STM32L011F4Ux, U4 THVD1400D, U5 SIP32434

Commit message: JLC order ready
Parts:
- R11: now fitted; now in the parts list
Changed lines of the file:
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@@
 		(body_style 1)
 		(exclude_from_sim no)
-		(in_bom no)
+		(in_bom yes)
 		(on_board yes)
 		(in_pos_files yes)
-		(dnp yes)
+		(dnp no)
 		(fields_autoplaced yes)
 		(property "Reference" "R11"
