File: life-bms/helios-bms-life.kicad_pcb (KiCad board)
At the start: 4 copper layers, 28.6 x 19 mm, 55 parts, among them J1 Outboard, J2 Debug, J3 Output, J4 Battery, Q1 SSM3J332R, Q2 Q_Dual_NMOS_PMOS_S1G1D2S2G2D1, Q3 PMOS, U1 TPSM861253, U2 BQ25306, U3 STM32L011F4Ux, U4 THVD1400D, U5 SIP32434

Commit message: BMS satellite boards ready, controller needs routing
Parts:
- added R24: 1M, Resistor_SMD:R_0402_1005Metric, B.Cu at (104.0, 80.5)
- added R25: 100k, Resistor_SMD:R_0402_1005Metric, B.Cu at (103.0, 80.5)
- D1: value TBD -> GSDH3005
- Q1: value SSM3J332R -> SSM6J507NU
- R13: value 500k -> 453k
- R14: value 100k -> 52.3k
Connections:
- Q2 pad 4: +12V -> VSYS
- Q3 pad 3: +12V -> VSYS
- R17 pad 1: +12V -> VSYS
- R20 pad 1: Net-(U5-OVP) -> /EN/UVLO
- R22 pad 2: Net-(U5-OVP) -> /EN/UVLO
Routing:
- net VSYS: track 35.7 -> 52.2 mm, vias 8 -> 9
- net +12V: track 48.2 -> 42.4 mm
- net /EN/UVLO: track 11.3 -> 16.5 mm
- net Net-(U5-OVP): track 8.54 -> 10.7 mm
- net GND: track 73.9 -> 75.2 mm

Commit message: JLC order ready
Routing:
- net VSYS: track 52.2 -> 51.2 mm
