File: lipo-bms/helios-bms-lipo.kicad_sch (KiCad schematic)
At the start: 36 parts, among them J1 Debug, J2 Output, J3 Outboard, J4 Battery, Q1 NMOS, U1 TPSM861253, U2 STM32L011F4Ux, U3 TPS22811, U6 THVD1400D

Commit message: satellite boards done
Parts:
- removed C11: 470u, Capacitor_THT:CP_Radial_D6.3mm_P2.50mm, symbol Device:C_Polarized
- removed C3, C9: 1u, Capacitor_SMD:C_0402_1005Metric, symbol Device:C_Small
- removed J2: Output, Connector_JST:JST_ZE_SM03B-ZESS-TB_1x03-1MP_P1.50mm_Horizontal, symbol Connector_Generic_MountingPin:Conn_01x02_MountingPin
- removed Q1: NMOS, Helios-BMS:SOT-1220_UDFN6B_TOS-L, symbol Helios-BMS:SSM6K388NU
- removed R1: TBD, Resistor_SMD:R_0402_1005Metric, symbol Device:R_Small_US
- removed R10: 150k, Resistor_SMD:R_0402_1005Metric, symbol Device:R_Small_US
- removed R11: 49.9k, Resistor_SMD:R_0402_1005Metric, symbol Device:R_Small_US
- removed R12: 10k, Resistor_SMD:R_0402_1005Metric, symbol Device:R_Small_US
- removed R9: 1k, Resistor_SMD:R_0402_1005Metric, symbol Device:R_Small_US
- removed U3: TPS22811, Helios-BMS:TPS22811, symbol Helios-BMS:TPS22811
- added C4, C6: 1u, Capacitor_SMD:C_0402_1005Metric, symbol Device:C_Small
- added C7: 10u, Capacitor_SMD:C_0603_1608Metric, symbol Device:C_Small
- added D1: Status, LED_SMD:LED_0402_1005Metric, symbol Device:LED_Small
- added D2: PG, LED_SMD:LED_0402_1005Metric, symbol Device:LED_Small
- added J3: Output, Connector_JST:JST_PH_S2B-PH-SM4-TB_1x02-1MP_P2.00mm_Horizontal, symbol Connector_Generic_MountingPin:Conn_01x02_MountingPin
- added R14: TBD, Resistor_SMD:R_0402_1005Metric, symbol Device:R_Small_US
- added R3, R7, R8: 10k, Resistor_SMD:R_0402_1005Metric, symbol Device:R_Small_US
- added U2: BQ25176M, Package_SON:WSON-8-1EP_2x2mm_P0.5mm_EP0.9x1.6mm_ThermalVias, symbol Helios-BMS:BQ25176M
- added U3: TPS22810DRV, Package_SON:WSON-6-1EP_2x2mm_P0.65mm_EP1x1.6mm, symbol Power_Management:TPS22810DRV
- C5: value 1.5n -> 1u
- J4: footprint Connector_JST:JST_ZE_SM03B-ZESS-TB_1x03-1MP_P1.50mm_Horizontal -> Connector_JST:JST_PH_S2B-PH-SM4-TB_1x02-1MP_P2.00mm_Horizontal
- R12: renamed from R7; value TBD -> 100k
- R13: renamed from R8; value TBD -> 330k
- R4: value 430k -> 35.7k
- R5: value 100k -> 10k
- R6: value 51k -> 510R
- renumbered C23 to C10, C8 to C3, C6 to C8, C4 to C9, J3 to J1, J1 to J2, R2 to R1, R24 to R10, R23 to R11, R3 to R2, R22 to R9, U2 to U4, U6 to U5
Connections:
- net BATT_ADC is gone; now on net PACK_ADC: U4.7 (PA4)
- net IMON is gone; now on net GATE: U4.9 (PA6)
- net +12V: now also C5.1, U2.1 (IN)
- net +BATT: now also J4.1 (Pin_1), R5.2, C4.1, C6.1, R3.2, R8.1, U2.8 (OUT), U3.6 (VIN); no longer J4.2 (Pin_2)
- net +VSW: now also C7.1, J3.1 (Pin_1), R14.1, U3.1 (VOUT)
- net GATE: now also R8.2, U3.5 (EN/UVLO); no longer U4.10 (PA7)
- net GND: now also J4.2 (Pin_2), R4.2, C4.2, C6.2, C7.2, J3.2 (Pin_2), R7.2, U2.4 (GND), U2.9 (GND), U3.3 (CT), U3.4 (GND), U3.7 (GND); no longer J4.1 (Pin_1)
- net PACK_ADC: now reaches R12.2, R13.1
- net EN/UVLO: no longer names the net of R5.1
- net EN/UVLO: now also D2.2 (A); no longer R4.2
- net VSYS: no longer names the net of R4.1
- net VSYS: now also U2.7 (VSET)
- net ~{EN}/OVLO: no longer names the net of R6.1
- net ~{EN}/OVLO: now also U2.2 (ISET); no longer R5.2
- new net: R7.1, U2.3 (BIAS)
- new net: D1.1 (K), U2.5 (STAT)
- new net: D2.1 (K), U2.6 (~{PG})
- new net: R14.2, U3.2 (QOD)
- new net: D1.2 (A), R3.1
- no-connect marks 12 -> 14
Other:
- note added: "4.2V Cell Max ~ 0.762 ratio RT ~ 0.3125RB Actual = 0.767"
- note added: "Auto powers up/ keeps on when MCU tristates"
- note added: "Battery Charger"
- note added: "Battery Voltage Monitoring"
- note added: "I_CHG = 600mA R_ISET = 300A*ohm/I_CHG = 500ohm -> 510ohm Acutal: 588mA"
- note added: "Table7-1 35.7kohm = 4.15V cutoff"
- note removed: "4.8V PGTH Eq. 13: 4.8V = 1.2V (Rtop + Rbot)/Rbot -> 4 = Rtop+Rbot/Rbot Rtop = 150k, Rbot = 50k 4.8V/(Rtop + Rbot) = 24uA >20x than PGTH leakage current 49.9k for sourcing reasons"
- note removed: "5ms rise time (to 12V): SR = 12V/5ms = 2.4V/ms Eq. 10: 3300/(2.4 V/ms) = 1375pF ~ 1500pF -> 2.2V/ms 2.2V/ms = 5.5ms"
- note removed: "Assume 0.5A load @ 6V for 6ms: (switching time) F = (0.5A * 15ms)/6V = 500uF ~ 470uF Gets better with less current or higher voltage Inrush(mA) = 470uF * 2.2V/ms = 1.034A PDinrush(W) = 0.5 * 12V * 1.034A = 6.204W That dissipated power is tolerable for ~100ms, much more than the ~6ms of inrush time expected"
- note removed: "Battery Cell Voltage Monitoring"
- note removed: "Close enough to reference design value. Should give 0.5V for ~5.2A."
- note removed: "MCU Enable Circuit Auto powers up/ keeps on when MCU tristates"
- note removed: "OVLO ~ 13.2V (ground power) UVLO ~ 4.6V (2.3V/cell) Values are close enough."
- moved on the sheet: C10, C8, C9, H1, H2, J1, J2, R10, R11, R12, R13, R9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

Commit message: JLC order ready
Parts:
- R10: now fitted; now in the parts list
- R3, R5: value 10k -> 300R
Changed lines of the file:
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@@
 		(body_style 1)
 		(exclude_from_sim no)
-		(in_bom no)
-		(on_board yes)
-		(in_pos_files yes)
-		(dnp yes)
+		(in_bom yes)
+		(on_board yes)
+		(in_pos_files yes)
+		(dnp no)
 		(fields_autoplaced yes)
 		(property "Reference" "R10"
@@
 			)
 		)
-		(property "Value" "10k"
+		(property "Value" "300R"
 			(at 132.588 29.718 90)
 			(show_name no)
@@
 			)
 		)
-		(property "Value" "10k"
+		(property "Value" "300R"
 			(at 132.588 42.672 90)
 			(show_name no)
