File: umbilical-controller/umbilical-controller.kicad_sch (KiCad schematic)
At the start: 35 parts, among them J1 RJ45, J2 RJ45, J3 Power In, J4 USB_C_Receptacle_USB2.0_16P, SW1 RESET, SW2 BOOT, U1 USBLC6-2SC6, U2 LM66100DCK, U3 LM66100DCK, U4 TPS62A01DRLR, U5 TPS56224, U6 ESP32-C6-MINI-1

Commit message: umbilical controller done
Parts:
- added H1, H2, H3, H4: MountingHole_Pad_MP, MountingHole:MountingHole_4.3mm_M4_ISO7380_Pad_TopBottom, symbol Mechanical:MountingHole_Pad
Connections:
- net GND: now also H1.1, H2.1, H3.1, H4.1
- net STATE1: now reaches U6.12 (IO0)
- net STATE2: now reaches U6.13 (IO1)
- no-connect marks 15 -> 11
Other:
- note added: "Todo:"
- note removed: "Todo: - Route"
