File: umbilical-controller/umbilical-controller.kicad_pcb (KiCad board)
At the start: 2 copper layers, 65 parts, among them J1 RJ45, J2 RJ45, J3 Power In, J4 USB_C_Receptacle_USB2.0_16P, SW1 RESET, SW2 BOOT, U1 USBLC6-2SC6, U10 SIP32434, U2 LM66100DCK, U3 LM66100DCK, U4 TPS62A01DRLR, U5 TPS56224, U6 ESP32-C6-MINI-1, U7 SIP32434, U8 THVD1400D, U9 THVD1400D

Commit message: umbilical controller done
Parts:
- added H1: MountingHole_Pad_MP, MountingHole:MountingHole_4.3mm_M4_ISO7380_Pad_TopBottom, F.Cu at (192.5, 80.0)
- added H2: MountingHole_Pad_MP, MountingHole:MountingHole_4.3mm_M4_ISO7380_Pad_TopBottom, F.Cu at (127.5, 80.0)
- added H3: MountingHole_Pad_MP, MountingHole:MountingHole_4.3mm_M4_ISO7380_Pad_TopBottom, F.Cu at (127.5, 120.0)
- added H4: MountingHole_Pad_MP, MountingHole:MountingHole_4.3mm_M4_ISO7380_Pad_TopBottom, F.Cu at (192.5, 120.0)
- moved J3 127.7 mm to (191.3, 112.5), turned to 90 degrees
- moved R2 114.3 mm to (180.7, 107.5), turned to 90 degrees
- moved R1 110.8 mm to (180.7, 110.6), turned to 90 degrees
- moved C6 101.9 mm to (173.3, 119.3)
- moved C8 101.0 mm to (176.4, 122.3), turned to 90 degrees
- moved J4 98.8 mm to (141.6, 121.3)
- moved C10 97.8 mm to (173.3, 117.5)
- moved R6 94.8 mm to (125.0, 110.8)
- moved R11 94.5 mm to (178.0, 119.2), turned to 90 degrees
- moved R10 94.4 mm to (178.0, 122.3), turned to 90 degrees
- moved C1 93.7 mm to (125.0, 112.3), turned to 180 degrees
- moved R5 90.0 mm to (135.6, 96.3), turned to 180 degrees
- moved R7 89.9 mm to (173.3, 120.9)
- moved C2 89.2 mm to (179.9, 118.0), turned to -90 degrees
- moved U5 88.9 mm to (175.8, 118.2), turned to -90 degrees
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Connections:
- R17 pad 1: /Load Switch2/SW_PG -> /STATE2
- R29 pad 1: /Load Switch1/SW_PG -> /STATE1
- U10 pad 8: /Load Switch1/SW_PG -> /STATE1
- U6 pad 12: unconnected-(U6-IO0-Pad12) -> /STATE1
- U6 pad 13: unconnected-(U6-IO1-Pad13) -> /STATE2
- U7 pad 8: /Load Switch2/SW_PG -> /STATE2
Routing:
- net GND: track 0.00 -> 188.3 mm, vias 0 -> 75
- net +12V: track 0.00 -> 148.5 mm, vias 0 -> 11
- net +3.3V: track 0.00 -> 104.2 mm, vias 0 -> 7
- net /DE1: track 0.00 -> 64.8 mm
- net /TX1: track 0.00 -> 63.9 mm, vias 0 -> 2
- net /RX1: track 0.00 -> 61.3 mm, vias 0 -> 2
- net /VMON: track 0.00 -> 52.9 mm, vias 0 -> 2
- net /IMON1: track 0.00 -> 49.3 mm, vias 0 -> 2
- net /GATE1: track 0.00 -> 44.2 mm, vias 0 -> 3
- net /STATE1: track 0.00 -> 42.9 mm, vias 0 -> 3
- net +5VP: track 0.00 -> 42.5 mm, vias 0 -> 2
- net VBUS: track 0.00 -> 31.0 mm
- net /DE2: track 0.00 -> 26.9 mm, vias 0 -> 2
- net /TX2: track 0.00 -> 23.2 mm, vias 0 -> 2
- net /IMON2: track 0.00 -> 22.3 mm, vias 0 -> 2
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- added copper zone on B.Cu, net GND
- added copper zone on F.Cu, net GND
Other:
- board outline added: 75 x 50 mm
- board text added: "+"
- board text added: "Enable"
- board text added: "GND"
- board text added: "Helios Umbilical Control Board"
- board text added: "Nic DeBruin KV0R 2026"
- board text added: "Port 1"
- board text added: "Port 2"
- board text added: "Power In +12V"
- board text added: "Reset"
- board text added: "todo: - routing"

Commit message: JLC order ready
Parts:
- C11, C13, C16, C18: footprint Capacitor_SMD:C_0805_2012Metric -> Capacitor_SMD:C_0603_1608Metric
Routing:
- net +12V: track 148.5 -> 152.4 mm
